File: _saved_VCF-VCA-SIP.sch (KiCad schematic (older format))
At the start: 44 parts, among them P1 CONN_10, Q1 BC857BS, U1 LM13700, U2 TL074-, U3 LM13700, U4 LM13700, U5 TL072-

Commit message: probably going to give up on this layout. What a pain
Parts:
- removed U2: TL074-, github-smd:TSSOP-14, symbol TL074-
- removed U4: LM13700, synth:SO16-JRL, symbol LM13700
- added U2, U4: TL072-, MyModules:TSSOP8-JRL, symbol TL072-
- added U5: LM13700, MyModules:SOIC16-12-JRL, symbol LM13700
- C1, C2, C3, C4, C5, C6, C7: footprint synth:SM0603-JRL -> MyModules:SM0603-C-JRL
- Q1: footprint synth:SOT363-JRL -> MyModules:SOT363-JRL
- R1, R10, R11, R12, R13, R14, R15, R16, R17, R18, R19, R2, R20, R21, R22, R23, R24, R25, R26, R27, R28, R3, R30, R4, R5, R6, R7, R8, R9: footprint synth:SM0603-JRL -> MyModules:SM0603-R-JRL
- R29: footprint github-smd:SMD-0805 -> MyModules:SM0805-HAND
- U1, U3: footprint synth:SO16-JRL -> MyModules:SOIC16-12-JRL
- U6: renamed from U5; footprint synth:TSSOP8-JRL -> MyModules:TSSOP8-JRL
Connections:
- net +VCC: now also U2.8 (V+), U4.8 (V+), U5.11 (V+)
- net -VCC: now also U2.4 (V-), U4.4 (V-), U5.6 (V-)
- net GND: now also U6.5 (+); no longer U6.3 (+)
- net RES_CTRL: now also U5.16
- net VCA_CTRL: now also U5.1
- net VCA_OUT: now also U6.1, U6.2 (-); no longer U6.6 (-), U6.7
- net VCF_OUT: now also U4.6 (-), U4.7
- net at R3.2, R4.2, R5.2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: now also U5.12
- net at C2.1, U1.5: now also U2.3 (+)
- net at R5.1, R7.2: now also U2.1, U2.2 (-)
- net at C3.1, U1.12: now also U2.5 (+)
- net at R11.2, R9.1: now also U2.6 (-), U2.7
- net at R11.1, R12.2, R13.2: now also U3.4 (-); no longer U3.13 (-)
- net at U3.12: now also C5.1, U4.5 (+); no longer C4.1
- net at U3.16: now also R18.1; no longer R14.1
- net at R13.1, R15.2: now also U4.1, U4.2 (-)
- net at R15.1, R16.2, R17.2: now also U3.13 (-); no longer U3.4 (-)
- net at U3.1: now also R14.1; no longer R18.1
- net at U3.5: now also C4.1, U4.3 (+); no longer C5.1
- net at R20.1, R22.2: now also U5.13 (-)
- net at R21.1, R27.2: now also U5.14 (+)
- net at R25.1: now also U5.3 (+)
- net at R23.1, R24.1: now also U5.4 (-)
- net at C6.1, R26.1: now also U6.3 (+), U5.5; no longer U6.5 (+)
- net at C1.2, Q1.6 (C1), R1.1: now also U6.6 (-); no longer U6.2 (-)
- net at C1.1, R2.2: now also U6.7; no longer U6.1
Other:
- moved on the sheet: U3A, U3B, U6A, U6B
