File: VCF-VCA-SIP.kicad_pcb (KiCad board)
At the start: 2 copper layers, 42 x 18 mm, 44 parts, among them P1 CONN_10, Q1 BC857BS, U1 LM13700, U2 TL074-, U3 LM13700, U4 LM13700, U5 TL072-

Commit message: bah, more hopelessness
Parts:
- R14, R18: moved to B.Cu
- moved C1 9.56 mm to (128.5, 89.9), turned to 270 degrees
- moved R10 8.28 mm to (114.8, 85.2), turned to 90 degrees
- moved R26 7.85 mm to (117.0, 89.8), turned to 90 degrees
- moved R14 7.77 mm to (133.5, 94.0), turned to 90 degrees
- moved R2 6.98 mm to (124.5, 89.8)
- moved R18 6.46 mm to (133.5, 86.1), turned to 270 degrees
- moved U5 6.17 mm to (122.0, 86.8), turned to 270 degrees
- moved R1 5.77 mm to (126.5, 89.9), turned to 90 degrees
- moved C6 5.15 mm to (115.1, 89.8), turned to 90 degrees
- moved R29 3.51 mm to (119.5, 92.2), turned to 0 degrees
- moved R6 2.29 mm to (115.0, 92.9)
- moved Q1 2.14 mm to (120.8, 89.8), turned to 270 degrees
- moved U4 1.19 mm to (106.6, 90.1), turned to 270 degrees
Connections:
- U5 pad 1: VCA_OUT -> Net-(C1-Pad1)
- U5 pad 2: VCA_OUT -> Net-(C1-Pad2)
- U5 pad 3: Net-(C6-Pad1) -> GND
- U5 pad 5: GND -> Net-(C6-Pad1)
- U5 pad 6: Net-(C1-Pad2) -> VCA_OUT
- U5 pad 7: Net-(C1-Pad1) -> VCA_OUT
Routing:
- net VCA_OUT: track 2.87 -> 38.7 mm
- net Iabc: track 0.00 -> 21.1 mm
- net +VCC: track 42.0 -> 23.9 mm, vias 2 -> 1
- net -VCC: track 56.7 -> 46.1 mm, vias 3 -> 2
- net Net-(C6-Pad1): track 18.4 -> 12.1 mm
- net Net-(R14-Pad1): track 0.80 -> 6.67 mm, vias 0 -> 1
- net Net-(R18-Pad1): track 0.80 -> 6.20 mm, vias 0 -> 1
- net Net-(C1-Pad1): track 11.7 -> 15.2 mm
- net Net-(R3-Pad2): track 26.9 -> 23.8 mm, vias 1 -> 0
- net Net-(C1-Pad2): track 11.1 -> 14.1 mm
- net VCF_CTRL: track 13.3 -> 11.1 mm
- net GND: track 0.00 -> 1.75 mm, vias 0 -> 1
- net Net-(C4-Pad1): track 14.1 -> 14.8 mm
- net Net-(Q1-Pad1): track 6.42 -> 5.72 mm
