File: VCF-VCA-SIP.sch (KiCad schematic (older format))
At the start: 45 parts, among them P1 CONN_10, Q1 BC857BS, U1 LM13700, U2 TL072-, U3 LM13700, U4 TL072-, U5 LM13700, U6 TL072-

Commit message: rearrange components and reroute
Connections:
- net GND: now also U6.5 (+); no longer U6.3 (+)
- net VCA_OUT: now also U6.1, U6.2 (-); no longer U6.6 (-), U6.7
- net at C6.1, R26.1, U5.12: now also U6.3 (+); no longer U6.5 (+)
- net at C1.2, Q1.6 (C1), R1.1: now also U6.6 (-); no longer U6.2 (-)
- net at C1.1, R2.2: now also U6.7; no longer U6.1
Other:
- moved on the sheet: U6A, U6B
Changed lines of the file:
@@
 L TL072- U6
 U 2 1 52F068F8
-P 11100 2075
-F 0 "U6" H 11050 2275 60  0000 L CNN
-F 1 "TL072-" H 11050 1825 60  0000 L CNN
-F 2 "MyModules:TSSOP8-JRL" H 11100 2075 60  0001 C CNN
-F 3 "~" H 11100 2075 60  0000 C CNN
-	2    11100 2075
+P 16800 3375
+F 0 "U6" H 16750 3575 60  0000 L CNN
+F 1 "TL072-" H 16750 3125 60  0000 L CNN
+F 2 "MyModules:TSSOP8-JRL" H 16800 3375 60  0001 C CNN
+F 3 "~" H 16800 3375 60  0000 C CNN
+	2    16800 3375
 	1    0    0    -1
 $EndComp
@@
 L TL072- U6
 U 1 1 52F070C4
-P 16800 3375
-F 0 "U6" H 16750 3575 60  0000 L CNN
-F 1 "TL072-" H 16750 3125 60  0000 L CNN
-F 2 "MyModules:TSSOP8-JRL" H 16800 3375 60  0001 C CNN
-F 3 "~" H 16800 3375 60  0000 C CNN
-	1    16800 3375
+P 11100 2075
+F 0 "U6" H 11050 2275 60  0000 L CNN
+F 1 "TL072-" H 11050 1825 60  0000 L CNN
+F 2 "MyModules:TSSOP8-JRL" H 11100 2075 60  0001 C CNN
+F 3 "~" H 11100 2075 60  0000 C CNN
+	1    11100 2075
 	1    0    0    -1
 $EndComp
@@
 L +VCC #PWR025
 U 1 1 52F070CA
-P 16700 2975
-F 0 "#PWR025" H 16700 3075 30  0001 C CNN
-F 1 "+VCC" H 16675 3250 60  0000 C CNN
-F 2 "~" H 16700 2975 60  0000 C CNN
-F 3 "~" H 16700 2975 60  0000 C CNN
-	1    16700 2975
+P 11000 1675
+F 0 "#PWR025" H 11000 1775 30  0001 C CNN
+F 1 "+VCC" H 10975 1950 60  0000 C CNN
+F 2 "~" H 11000 1675 60  0000 C CNN
+F 3 "~" H 11000 1675 60  0000 C CNN
+	1    11000 1675
 	1    0    0    -1
 $EndComp
@@
 L -VCC #PWR026
 U 1 1 52F070D0
-P 16700 3775
-F 0 "#PWR026" H 16700 3875 30  0001 C CNN
-F 1 "-VCC" H 16675 4050 60  0000 C CNN
-F 2 "~" H 16700 3775 60  0000 C CNN
-F 3 "~" H 16700 3775 60  0000 C CNN
-	1    16700 3775
+P 11000 2475
+F 0 "#PWR026" H 11000 2575 30  0001 C CNN
+F 1 "-VCC" H 10975 2750 60  0000 C CNN
+F 2 "~" H 11000 2475 60  0000 C CNN
+F 3 "~" H 11000 2475 60  0000 C CNN
+	1    11000 2475
 	-1   0    0    1
 $EndComp
@@
 	2400 6525 2150 6525
 Wire Wire Line
-	2150 5775 2150 6625
-Wire Wire Line
-	1750 6825 2400 6825
+	2150 5775 2150 6525
+Wire Wire Line
+	2150 6525 2150 6625
+Wire Wire Line
+	1750 6825 1800 6825
+Wire Wire Line
+	1800 6825 1900 6825
+Wire Wire Line
+	1900 6825 2250 6825
+Wire Wire Line
+	2250 6825 2400 6825
 Connection ~ 1800 6825
 Wire Wire Line
@@
 	1900 7475 1900 7625
 Wire Wire Line
-	950  6825 1400 6825
+	950  6825 1150 6825
+Wire Wire Line
+	1150 6825 1400 6825
 Wire Wire Line
 	1150 6825 1150 6275
@@
 	3850 5675 4850 5675
 Wire Wire Line
-	4850 5675 4850 8025
-Wire Wire Line
-	3500 6675 3850 6675
+	4850 5675 4850 6575
+Wire Wire Line
+	4850 6575 4850 6825
+Wire Wire Line
+	4850 6825 4850 8025
+Wire Wire Line
+	3500 6675 3650 6675
+Wire Wire Line
+	3650 6675 3850 6675
 Wire Wire Line
 	3650 7475 3650 7625
@@
 Connection ~ 3650 6675
 Wire Wire Line
-	2250 6825 2250 8375
+	2250 6825 2250 8025
+Wire Wire Line
+	2250 8025 2250 8375
 Wire Wire Line
 	2250 8025 3550 8025
@@
 	5900 6525 5900 6625
 Wire Wire Line
-	5500 6825 6150 6825
+	5500 6825 5650 6825
+Wire Wire Line
+	5650 6825 6000 6825
+Wire Wire Line
+	6000 6825 6150 6825
 Wire Wire Line
 	5650 7075 5650 6825
@@
 	5650 7475 5650 7625
 Wire Wire Line
-	7250 6675 7600 6675
+	7250 6675 7400 6675
+Wire Wire Line
+	7400 6675 7600 6675
 Wire Wire Line
 	7400 7475 7400 7625
@@
 	9650 6525 9650 6625
 Wire Wire Line
-	9250 6825 9900 6825
+	9250 6825 9400 6825
+Wire Wire Line
+	9400 6825 9750 6825
+Wire Wire Line
+	9750 6825 9900 6825
 Wire Wire Line
 	9400 7075 9400 6825
@@
 	11350 5750 12350 5750
 Wire Wire Line
-	12350 5750 12350 8025
-Wire Wire Line
-	11000 6675 11350 6675
+	12350 5750 12350 6575
+Wire Wire Line
+	12350 6575 12350 6825
+Wire Wire Line
+	12350 6825 12350 8025
+Wire Wire Line
+	11000 6675 11150 6675
+Wire Wire Line
+	11150 6675 11350 6675
 Wire Wire Line
 	11150 7475 11150 7625
@@
 	13400 6525 13400 6625
 Wire Wire Line
-	13000 6825 13650 6825
+	13000 6825 13150 6825
+Wire Wire Line
+	13150 6825 13500 6825
+Wire Wire Line
+	13500 6825 13650 6825
 Wire Wire Line
 	13150 7075 13150 6825
@@
 	15100 6175 16100 6175
 Wire Wire Line
-	16100 6175 16100 8025
-Wire Wire Line
-	14750 6675 15100 6675
+	16100 6175 16100 6575
+Wire Wire Line
+	16100 6575 16100 6825
+Wire Wire Line
+	16100 6825 16100 8025
+Wire Wire Line
+	14750 6675 14900 6675
+Wire Wire Line
+	14900 6675 15100 6675
 Wire Wire Line
 	14900 7475 14900 7625
@@
 Connection ~ 13500 6825
 Wire Wire Line
-	15200 8025 16300 8025
+	15200 8025 16100 8025
+Wire Wire Line
+	16100 8025 16300 8025
 Connection ~ 16100 6575
 Wire Wire Line
@@
 Connection ~ 16100 8025
 Wire Wire Line
-	17350 6525 17450 6525
-Wire Wire Line
-	3350 5425 14850 5425
+	17350 6525 17400 6525
+Wire Wire Line
+	17400 6525 17450 6525
+Wire Wire Line
+	3350 5425 7100 5425
+Wire Wire Line
+	7100 5425 10850 5425
+Wire Wire Line
+	10850 5425 14600 5425
+Wire Wire Line
+	14600 5425 14850 5425
 Connection ~ 7100 5425
 Connection ~ 10850 5425
@@
 	7600 6175 8600 6175
 Wire Wire Line
-	8600 6175 8600 8025
-Wire Wire Line
-	16750 6825 17450 6825
+	8600 6175 8600 6575
+Wire Wire Line
+	8600 6575 8600 6825
+Wire Wire Line
+	8600 6825 8600 8025
+Wire Wire Line
+	16750 6825 16950 6825
+Wire Wire Line
+	16950 6825 17450 6825
 Wire Wire Line
 	16950 6525 16950 6625
@@
 Connection ~ 17400 6525
 Wire Wire Line
-	7750 2325 8500 2325
+	7750 2325 8350 2325
+Wire Wire Line
+	8350 2325 8500 2325
 Wire Wire Line
 	8500 2025 8050 2025
@@
 	8050 3075 8050 3225
 Wire Wire Line
-	8050 3225 8350 3225
+	8050 3225 8200 3225
+Wire Wire Line
+	8200 3225 8350 3225
 Wire Wire Line
 	8350 3225 8350 3075
@@
 Connection ~ 8200 3225
 Wire Wire Line
-	7175 2325 7350 2325
+	7175 2325 7300 2325
+Wire Wire Line
+	7300 2325 7350 2325
 Wire Wire Line
 	9450 2125 9450 1425
@@
 	9450 1425 9700 1425
 Wire Wire Line
-	9600 2175 10600 2175
-Wire Wire Line
-	10600 1975 10600 1675
-Wire Wire Line
-	10600 1675 11600 1675
-Wire Wire Line
-	11600 1675 11600 2075
+	9600 2175 9900 2175
+Wire Wire Line
+	9900 2175 10450 2175
+Wire Wire Line
+	10450 2175 10600 2175
+Wire Wire Line
+	10600 1975 10600 1275
+Wire Wire Line
+	10600 1275 11600 1275
+Wire Wire Line
+	11600 1275 11600 2075
 Wire Wire Line
 	11600 2075 11850 2075
@@
 	9900 3025 9900 3225
 Wire Wire Line
-	9900 3225 10450 3225
+	9900 3225 10200 3225
+Wire Wire Line
+	10200 3225 10450 3225
 Wire Wire Line
 	10450 3225 10450 3025
@@
 	15200 1775 15200 1925
 Wire Wire Line
-	15750 2025 15950 2025
+	15750 2025 15850 2025
+Wire Wire Line
+	15850 2025 15950 2025
 Wire Wire Line
 	15850 2125 15850 2025
 Connection ~ 15850 2025
 Wire Wire Line
-	15850 2525 15850 2625
+	15850 2525 15850 2575
+Wire Wire Line
+	15850 2575 15850 2625
 Wire Wire Line
 	15850 2575 17300 2575
@@
 Connection ~ 15850 2575
 Wire Wire Line
-	15000 3275 16300 3275
-Wire Wire Line
-	15850 3025 15850 3475
+	15000 3275 15850 3275
+Wire Wire Line
+	15850 3275 16300 3275
+Wire Wire Line
+	15850 3025 15850 3275
+Wire Wire Line
+	15850 3275 15850 3475
 Connection ~ 15850 3275
 Wire Wire Line
@@
 	2800 2475 2400 2475
 Wire Wire Line
-	16300 1775 17150 1775
+	16300 1775 16875 1775
+Wire Wire Line
+	16875 1775 17150 1775
 Wire Notes Line
 	14700 875  17750 875
@@
 	1150 5025 1150 5250
 Wire Wire Line
-	1150 5650 1150 5875
+	1150 5650 1150 5775
+Wire Wire Line
+	1150 5775 1150 5875
 Wire Wire Line
 	1775 5775 2150 5775

Commit message: probably going to give up on this layout. What a pain
Connections:
- net RES_CTRL: now also U5.16; no longer U5.1
- net VCA_CTRL: now also U5.1; no longer U5.16
- net at R3.2, R4.2, R5.2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: now also U5.12; no longer U5.5
- net at R20.1, R22.2: now also U5.13 (-); no longer U5.4 (-)
- net at R21.1, R27.2: now also U5.14 (+); no longer U5.3 (+)
- net at R23.1, R24.1: now also U5.4 (-); no longer U5.13 (-)
- net at R25.1: now also U5.3 (+); no longer U5.14 (+)
- net at C6.1, R26.1, U6.3 (+): now also U5.5; no longer U5.12
Other:
- moved on the sheet: U5A, U5B
Changed lines of the file:
@@
 L +VCC #PWR017
 U 1 1 52F05AC4
-P 8950 1775
-F 0 "#PWR017" H 8950 1875 30  0001 C CNN
-F 1 "+VCC" H 8925 2050 60  0000 C CNN
-F 2 "~" H 8950 1775 60  0000 C CNN
-F 3 "~" H 8950 1775 60  0000 C CNN
-	1    8950 1775
+P 17900 6275
+F 0 "#PWR017" H 17900 6375 30  0001 C CNN
+F 1 "+VCC" H 17875 6550 60  0000 C CNN
+F 2 "~" H 17900 6275 60  0000 C CNN
+F 3 "~" H 17900 6275 60  0000 C CNN
+	1    17900 6275
 	1    0    0    -1
 $EndComp
@@
 L -VCC #PWR018
 U 1 1 52F05ACA
-P 8950 2575
-F 0 "#PWR018" H 8950 2675 30  0001 C CNN
-F 1 "-VCC" H 8925 2850 60  0000 C CNN
-F 2 "~" H 8950 2575 60  0000 C CNN
-F 3 "~" H 8950 2575 60  0000 C CNN
-	1    8950 2575
+P 17900 7075
+F 0 "#PWR018" H 17900 7175 30  0001 C CNN
+F 1 "-VCC" H 17875 7350 60  0000 C CNN
+F 2 "~" H 17900 7075 60  0000 C CNN
+F 3 "~" H 17900 7075 60  0000 C CNN
+	1    17900 7075
 	-1   0    0    1
 $EndComp
@@
 	2400 6525 2150 6525
 Wire Wire Line
-	2150 5775 2150 6525
-Wire Wire Line
-	2150 6525 2150 6625
-Wire Wire Line
-	1750 6825 1800 6825
-Wire Wire Line
-	1800 6825 1900 6825
-Wire Wire Line
-	1900 6825 2250 6825
-Wire Wire Line
-	2250 6825 2400 6825
+	2150 5775 2150 6625
+Wire Wire Line
+	1750 6825 2400 6825
 Connection ~ 1800 6825
 Wire Wire Line
@@
 	1900 7475 1900 7625
 Wire Wire Line
-	950  6825 1150 6825
-Wire Wire Line
-	1150 6825 1400 6825
+	950  6825 1400 6825
 Wire Wire Line
 	1150 6825 1150 6275
@@
 	3850 5675 4850 5675
 Wire Wire Line
-	4850 5675 4850 6575
-Wire Wire Line
-	4850 6575 4850 6825
-Wire Wire Line
-	4850 6825 4850 8025
-Wire Wire Line
-	3500 6675 3650 6675
-Wire Wire Line
-	3650 6675 3850 6675
+	4850 5675 4850 8025
+Wire Wire Line
+	3500 6675 3850 6675
 Wire Wire Line
 	3650 7475 3650 7625
@@
 Connection ~ 3650 6675
 Wire Wire Line
-	2250 6825 2250 8025
-Wire Wire Line
-	2250 8025 2250 8375
+	2250 6825 2250 8375
 Wire Wire Line
 	2250 8025 3550 8025
@@
 	5900 6525 5900 6625
 Wire Wire Line
-	5500 6825 5650 6825
-Wire Wire Line
-	5650 6825 6000 6825
-Wire Wire Line
-	6000 6825 6150 6825
+	5500 6825 6150 6825
 Wire Wire Line
 	5650 7075 5650 6825
@@
 	5650 7475 5650 7625
 Wire Wire Line
-	7250 6675 7400 6675
-Wire Wire Line
-	7400 6675 7600 6675
+	7250 6675 7600 6675
 Wire Wire Line
 	7400 7475 7400 7625
@@
 	9650 6525 9650 6625
 Wire Wire Line
-	9250 6825 9400 6825
-Wire Wire Line
-	9400 6825 9750 6825
-Wire Wire Line
-	9750 6825 9900 6825
+	9250 6825 9900 6825
 Wire Wire Line
 	9400 7075 9400 6825
@@
 	11350 5750 12350 5750
 Wire Wire Line
-	12350 5750 12350 6575
-Wire Wire Line
-	12350 6575 12350 6825
-Wire Wire Line
-	12350 6825 12350 8025
-Wire Wire Line
-	11000 6675 11150 6675
-Wire Wire Line
-	11150 6675 11350 6675
+	12350 5750 12350 8025
+Wire Wire Line
+	11000 6675 11350 6675
 Wire Wire Line
 	11150 7475 11150 7625
@@
 	13400 6525 13400 6625
 Wire Wire Line
-	13000 6825 13150 6825
-Wire Wire Line
-	13150 6825 13500 6825
-Wire Wire Line
-	13500 6825 13650 6825
+	13000 6825 13650 6825
 Wire Wire Line
 	13150 7075 13150 6825
@@
 	15100 6175 16100 6175
 Wire Wire Line
-	16100 6175 16100 6575
-Wire Wire Line
-	16100 6575 16100 6825
-Wire Wire Line
-	16100 6825 16100 8025
-Wire Wire Line
-	14750 6675 14900 6675
-Wire Wire Line
-	14900 6675 15100 6675
+	16100 6175 16100 8025
+Wire Wire Line
+	14750 6675 15100 6675
 Wire Wire Line
 	14900 7475 14900 7625
@@
 Connection ~ 13500 6825
 Wire Wire Line
-	15200 8025 16100 8025
-Wire Wire Line
-	16100 8025 16300 8025
+	15200 8025 16300 8025
 Connection ~ 16100 6575
 Wire Wire Line
@@
 Connection ~ 16100 8025
 Wire Wire Line
-	17350 6525 17400 6525
-Wire Wire Line
-	17400 6525 17450 6525
-Wire Wire Line
-	3350 5425 7100 5425
-Wire Wire Line
-	7100 5425 10850 5425
-Wire Wire Line
-	10850 5425 14600 5425
-Wire Wire Line
-	14600 5425 14850 5425
+	17350 6525 17450 6525
+Wire Wire Line
+	3350 5425 14850 5425
 Connection ~ 7100 5425
 Connection ~ 10850 5425
@@
 	7600 6175 8600 6175
 Wire Wire Line
-	8600 6175 8600 6575
-Wire Wire Line
-	8600 6575 8600 6825
-Wire Wire Line
-	8600 6825 8600 8025
-Wire Wire Line
-	16750 6825 16950 6825
-Wire Wire Line
-	16950 6825 17450 6825
+	8600 6175 8600 8025
+Wire Wire Line
+	16750 6825 17450 6825
 Wire Wire Line
 	16950 6525 16950 6625
@@
 Connection ~ 17400 6525
 Wire Wire Line
-	7750 2325 8350 2325
-Wire Wire Line
-	8350 2325 8500 2325
+	7750 2325 8500 2325
 Wire Wire Line
 	8500 2025 8050 2025
@@
 	8050 3075 8050 3225
 Wire Wire Line
-	8050 3225 8200 3225
-Wire Wire Line
-	8200 3225 8350 3225
+	8050 3225 8350 3225
 Wire Wire Line
 	8350 3225 8350 3075
@@
 Connection ~ 8200 3225
 Wire Wire Line
-	7175 2325 7300 2325
-Wire Wire Line
-	7300 2325 7350 2325
+	7175 2325 7350 2325
 Wire Wire Line
 	9450 2125 9450 1425
@@
 	9450 1425 9700 1425
 Wire Wire Line
-	9600 2175 9900 2175
-Wire Wire Line
-	9900 2175 10450 2175
-Wire Wire Line
-	10450 2175 10600 2175
+	9600 2175 10600 2175
 Wire Wire Line
 	10600 1975 10600 1275
@@
 	9900 3025 9900 3225
 Wire Wire Line
-	9900 3225 10200 3225
-Wire Wire Line
-	10200 3225 10450 3225
+	9900 3225 10450 3225
 Wire Wire Line
 	10450 3225 10450 3025
@@
 	15200 1775 15200 1925
 Wire Wire Line
-	15750 2025 15850 2025
-Wire Wire Line
-	15850 2025 15950 2025
+	15750 2025 15950 2025
 Wire Wire Line
 	15850 2125 15850 2025
 Connection ~ 15850 2025
 Wire Wire Line
-	15850 2525 15850 2575
-Wire Wire Line
-	15850 2575 15850 2625
+	15850 2525 15850 2625
 Wire Wire Line
 	15850 2575 17300 2575
@@
 Connection ~ 15850 2575
 Wire Wire Line
-	15000 3275 15850 3275
-Wire Wire Line
-	15850 3275 16300 3275
-Wire Wire Line
-	15850 3025 15850 3275
-Wire Wire Line
-	15850 3275 15850 3475
+	15000 3275 16300 3275
+Wire Wire Line
+	15850 3025 15850 3475
 Connection ~ 15850 3275
 Wire Wire Line
@@
 	2800 2475 2400 2475
 Wire Wire Line
-	16300 1775 16875 1775
-Wire Wire Line
-	16875 1775 17150 1775
+	16300 1775 17150 1775
 Wire Notes Line
 	14700 875  17750 875
@@
 	1150 5025 1150 5250
 Wire Wire Line
-	1150 5650 1150 5775
-Wire Wire Line
-	1150 5775 1150 5875
+	1150 5650 1150 5875
 Wire Wire Line
 	1775 5775 2150 5775
@@
 L LM13700 U5
 U 1 1 56468C7F
+P 9100 2175
+F 0 "U5" H 9200 1975 60  0000 C CNN
+F 1 "LM13700" H 9000 2175 60  0000 C CNN
+F 2 "MyModules:SO16-JRL" H 9100 2175 60  0001 C CNN
+F 3 "" H 9100 2175 60  0000 C CNN
+	1    9100 2175
+	1    0    0    -1
+$EndComp
+$Comp
+L LM13700 U5
+U 2 1 56469641
 P 18050 6675
 F 0 "U5" H 18150 6475 60  0000 C CNN
@@
 F 2 "MyModules:SO16-JRL" H 18050 6675 60  0001 C CNN
 F 3 "" H 18050 6675 60  0000 C CNN
-	1    18050 6675
-	1    0    0    -1
-$EndComp
-$Comp
-L LM13700 U5
-U 2 1 56469641
-P 9100 2175
-F 0 "U5" H 9200 1975 60  0000 C CNN
-F 1 "LM13700" H 9000 2175 60  0000 C CNN
-F 2 "MyModules:SO16-JRL" H 9100 2175 60  0001 C CNN
-F 3 "" H 9100 2175 60  0000 C CNN
-	2    9100 2175
-	1    0    0    -1
-$EndComp
+	2    18050 6675
+	1    0    0    -1
+$EndComp

Commit message: last commit before checking out earlier version
Parts:
- U1, U3, U5: footprint MyModules:SO16-JRL -> MyModules:SOIC16-12-JRL
Changed lines of the file:
@@
 F 0 "U1" H 3100 6200 60  0000 C CNN
 F 1 "LM13700" H 3100 6300 60  0000 C CNN
-F 2 "MyModules:SO16-JRL" H 3000 6675 60  0001 C CNN
+F 2 "MyModules:SOIC16-12-JRL" H 3000 6675 60  0001 C CNN
 F 3 "~" H 3000 6675 60  0000 C CNN
 	1    3000 6675
@@
 F 0 "U1" H 6900 6350 60  0000 C CNN
 F 1 "LM13700" H 6900 6450 60  0000 C CNN
-F 2 "MyModules:SO16-JRL" H 6750 6675 60  0001 C CNN
+F 2 "MyModules:SOIC16-12-JRL" H 6750 6675 60  0001 C CNN
 F 3 "~" H 6750 6675 60  0000 C CNN
 	2    6750 6675
@@
 F 0 "U3" H 14400 6300 60  0000 C CNN
 F 1 "LM13700" H 14400 6400 60  0000 C CNN
-F 2 "MyModules:SO16-JRL" H 14250 6675 60  0001 C CNN
+F 2 "MyModules:SOIC16-12-JRL" H 14250 6675 60  0001 C CNN
 F 3 "~" H 14250 6675 60  0000 C CNN
 	2    14250 6675
@@
 F 0 "U3" H 10600 6300 60  0000 C CNN
 F 1 "LM13700" H 10600 6400 60  0000 C CNN
-F 2 "MyModules:SO16-JRL" H 10500 6675 60  0001 C CNN
+F 2 "MyModules:SOIC16-12-JRL" H 10500 6675 60  0001 C CNN
 F 3 "~" H 10500 6675 60  0000 C CNN
 	1    10500 6675
@@
 F 0 "U5" H 9200 1975 60  0000 C CNN
 F 1 "LM13700" H 9000 2175 60  0000 C CNN
-F 2 "MyModules:SO16-JRL" H 9100 2175 60  0001 C CNN
+F 2 "MyModules:SOIC16-12-JRL" H 9100 2175 60  0001 C CNN
 F 3 "" H 9100 2175 60  0000 C CNN
 	1    9100 2175
@@
 F 0 "U5" H 18150 6475 60  0000 C CNN
 F 1 "LM13700" H 17950 6675 60  0000 C CNN
-F 2 "MyModules:SO16-JRL" H 18050 6675 60  0001 C CNN
+F 2 "MyModules:SOIC16-12-JRL" H 18050 6675 60  0001 C CNN
 F 3 "" H 18050 6675 60  0000 C CNN
 	2    18050 6675
