File: VCF-VCA-SIP.sch (KiCad schematic (older format))
At the start: 45 parts, among them P1 CONN_10, Q1 BC857BS, U1 LM13700, U2 TL072-, U3 LM13700, U4 TL072-, U5 LM13700, U6 TL072-

Commit message: still struggling. about to go back to original layout
Parts:
- removed U2, U4: TL072-, MyModules:TSSOP8-JRL, symbol TL072-
- added U2: TL074-, Housings_SSOP:TSSOP-14_4.4x5mm_Pitch0.65mm, symbol TL074-
- renumbered U5 to U4, U6 to U5
Connections:
- net +VCC: now also U2.4 (V+)
- net -VCC: now also U2.11 (V-)
- net VCF_OUT: now also U2.8, U2.9 (-)
- net at U1.1: now also R10.1; no longer R6.1
- net at R3.2, R4.2, R5.2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: now also U1.13 (-); no longer U1.4 (-)
- net at U1.5: now also C3.1, U2.12 (+); no longer C2.1
- net at R5.1, R7.2: now also U2.1, U2.2 (-)
- net at R7.1, R8.2, R9.2: now also U1.4 (-); no longer U1.13 (-)
- net at U1.12: now also C2.1, U2.3 (+); no longer C3.1
- net at U1.16: now also R6.1; no longer R10.1
- net at R11.2, R9.1: now also U2.13 (-), U2.14
- net at R11.1, R12.2, R13.2: now also U3.13 (-); no longer U3.4 (-)
- net at U3.12: now also C4.1, U2.5 (+); no longer C5.1
- net at R15.1, R16.2, R17.2: now also U3.4 (-); no longer U3.13 (-)
- net at U3.16: now also R14.1; no longer R18.1
- net at U3.5: now also C5.1, U2.10 (+); no longer C4.1
- net at R13.1, R15.2: now also U2.6 (-), U2.7
- net at U3.1: now also R18.1; no longer R14.1
Other:
- moved on the sheet: U1A, U1B, U3A, U3B
Changed lines of the file:
@@
 L LM13700 U1
 U 1 1 52F056B5
-P 3000 6675
-F 0 "U1" H 3100 6200 60  0000 C CNN
-F 1 "LM13700" H 3100 6300 60  0000 C CNN
-F 2 "MyModules:SOIC16-12-JRL" H 3000 6675 60  0001 C CNN
-F 3 "~" H 3000 6675 60  0000 C CNN
-	1    3000 6675
+P 6750 6675
+F 0 "U1" H 6850 6200 60  0000 C CNN
+F 1 "LM13700" H 6850 6300 60  0000 C CNN
+F 2 "MyModules:SOIC16-12-JRL" H 6750 6675 60  0001 C CNN
+F 3 "~" H 6750 6675 60  0000 C CNN
+	1    6750 6675
 	1    0    0    -1
 $EndComp
@@
 L LM13700 U1
 U 2 1 52F059E4
-P 6750 6675
-F 0 "U1" H 6900 6350 60  0000 C CNN
-F 1 "LM13700" H 6900 6450 60  0000 C CNN
-F 2 "MyModules:SOIC16-12-JRL" H 6750 6675 60  0001 C CNN
-F 3 "~" H 6750 6675 60  0000 C CNN
-	2    6750 6675
+P 3000 6675
+F 0 "U1" H 3150 6350 60  0000 C CNN
+F 1 "LM13700" H 3150 6450 60  0000 C CNN
+F 2 "MyModules:SOIC16-12-JRL" H 3000 6675 60  0001 C CNN
+F 3 "~" H 3000 6675 60  0000 C CNN
+	2    3000 6675
 	1    0    0    -1
 $EndComp
@@
 L +VCC #PWR07
 U 1 1 52F05A08
-P 6600 6275
-F 0 "#PWR07" H 6600 6375 30  0001 C CNN
-F 1 "+VCC" H 6575 6550 60  0000 C CNN
-F 2 "~" H 6600 6275 60  0000 C CNN
-F 3 "~" H 6600 6275 60  0000 C CNN
-	1    6600 6275
+P 2850 6275
+F 0 "#PWR07" H 2850 6375 30  0001 C CNN
+F 1 "+VCC" H 2825 6550 60  0000 C CNN
+F 2 "~" H 2850 6275 60  0000 C CNN
+F 3 "~" H 2850 6275 60  0000 C CNN
+	1    2850 6275
 	1    0    0    -1
 $EndComp
@@
 L -VCC #PWR08
 U 1 1 52F05A0E
-P 6600 7075
-F 0 "#PWR08" H 6600 7175 30  0001 C CNN
-F 1 "-VCC" H 6575 7350 60  0000 C CNN
-F 2 "~" H 6600 7075 60  0000 C CNN
-F 3 "~" H 6600 7075 60  0000 C CNN
-	1    6600 7075
+P 2850 7075
+F 0 "#PWR08" H 2850 7175 30  0001 C CNN
+F 1 "-VCC" H 2825 7350 60  0000 C CNN
+F 2 "~" H 2850 7075 60  0000 C CNN
+F 3 "~" H 2850 7075 60  0000 C CNN
+	1    2850 7075
 	-1   0    0    1
 $EndComp
@@
 L LM13700 U3
 U 2 1 52F05A42
-P 14250 6675
-F 0 "U3" H 14400 6300 60  0000 C CNN
-F 1 "LM13700" H 14400 6400 60  0000 C CNN
-F 2 "MyModules:SOIC16-12-JRL" H 14250 6675 60  0001 C CNN
-F 3 "~" H 14250 6675 60  0000 C CNN
-	2    14250 6675
+P 10500 6675
+F 0 "U3" H 10650 6300 60  0000 C CNN
+F 1 "LM13700" H 10650 6400 60  0000 C CNN
+F 2 "MyModules:SOIC16-12-JRL" H 10500 6675 60  0001 C CNN
+F 3 "~" H 10500 6675 60  0000 C CNN
+	2    10500 6675
 	1    0    0    -1
 $EndComp
@@
 L +VCC #PWR012
 U 1 1 52F05A66
-P 14100 6275
-F 0 "#PWR012" H 14100 6375 30  0001 C CNN
-F 1 "+VCC" H 14075 6550 60  0000 C CNN
-F 2 "~" H 14100 6275 60  0000 C CNN
-F 3 "~" H 14100 6275 60  0000 C CNN
-	1    14100 6275
+P 10350 6275
+F 0 "#PWR012" H 10350 6375 30  0001 C CNN
+F 1 "+VCC" H 10325 6550 60  0000 C CNN
+F 2 "~" H 10350 6275 60  0000 C CNN
+F 3 "~" H 10350 6275 60  0000 C CNN
+	1    10350 6275
 	1    0    0    -1
 $EndComp
@@
 L -VCC #PWR013
 U 1 1 52F05A6C
-P 14100 7075
-F 0 "#PWR013" H 14100 7175 30  0001 C CNN
-F 1 "-VCC" H 14075 7350 60  0000 C CNN
-F 2 "~" H 14100 7075 60  0000 C CNN
-F 3 "~" H 14100 7075 60  0000 C CNN
-	1    14100 7075
+P 10350 7075
+F 0 "#PWR013" H 10350 7175 30  0001 C CNN
+F 1 "-VCC" H 10325 7350 60  0000 C CNN
+F 2 "~" H 10350 7075 60  0000 C CNN
+F 3 "~" H 10350 7075 60  0000 C CNN
+	1    10350 7075
 	-1   0    0    1
 $EndComp
@@
 L LM13700 U3
 U 1 1 52F05AA0
-P 10500 6675
-F 0 "U3" H 10600 6300 60  0000 C CNN
-F 1 "LM13700" H 10600 6400 60  0000 C CNN
-F 2 "MyModules:SOIC16-12-JRL" H 10500 6675 60  0001 C CNN
-F 3 "~" H 10500 6675 60  0000 C CNN
-	1    10500 6675
+P 14250 6675
+F 0 "U3" H 14350 6300 60  0000 C CNN
+F 1 "LM13700" H 14350 6400 60  0000 C CNN
+F 2 "MyModules:SOIC16-12-JRL" H 14250 6675 60  0001 C CNN
+F 3 "~" H 14250 6675 60  0000 C CNN
+	1    14250 6675
 	1    0    0    -1
 $EndComp
@@
 VCA_CTRL
 $Comp
-L TL072- U6
+L TL072- U5
 U 2 1 52F068F8
 P 16800 3375
-F 0 "U6" H 16750 3575 60  0000 L CNN
+F 0 "U5" H 16750 3575 60  0000 L CNN
 F 1 "TL072-" H 16750 3125 60  0000 L CNN
 F 2 "MyModules:TSSOP8-JRL" H 16800 3375 60  0001 C CNN
@@
 $EndComp
 $Comp
-L TL072- U6
+L TL072- U5
 U 1 1 52F070C4
 P 11100 2075
-F 0 "U6" H 11050 2275 60  0000 L CNN
+F 0 "U5" H 11050 2275 60  0000 L CNN
 F 1 "TL072-" H 11050 1825 60  0000 L CNN
 F 2 "MyModules:TSSOP8-JRL" H 11100 2075 60  0001 C CNN
@@
 NoConn ~ 6850 6375
 NoConn ~ 10600 6375
-NoConn ~ 14350 6375
+NoConn ~ 10600 6375
 NoConn ~ 9200 1875
 NoConn ~ 9200 1875
@@
 	7175 1900 7175 1925
 $Comp
-L TL072- U2
-U 1 1 564652C3
-P 4350 6575
-F 0 "U2" H 4300 6775 60  0000 L CNN
-F 1 "TL072-" H 4300 6325 60  0000 L CNN
-F 2 "MyModules:TSSOP8-JRL" H 4350 6575 60  0001 C CNN
-F 3 "" H 4350 6575 60  0000 C CNN
-	1    4350 6575
-	1    0    0    -1
-$EndComp
-$Comp
-L TL072- U2
-U 2 1 564654BE
-P 8100 6575
-F 0 "U2" H 8050 6775 60  0000 L CNN
-F 1 "TL072-" H 8050 6325 60  0000 L CNN
-F 2 "MyModules:TSSOP8-JRL" H 8100 6575 60  0001 C CNN
-F 3 "" H 8100 6575 60  0000 C CNN
-	2    8100 6575
-	1    0    0    -1
-$EndComp
-$Comp
-L TL072- U4
-U 1 1 564659EC
-P 11850 6575
-F 0 "U4" H 11800 6775 60  0000 L CNN
-F 1 "TL072-" H 11800 6325 60  0000 L CNN
-F 2 "MyModules:TSSOP8-JRL" H 11850 6575 60  0001 C CNN
-F 3 "" H 11850 6575 60  0000 C CNN
-	1    11850 6575
-	1    0    0    -1
-$EndComp
-$Comp
 L +VCC #PWR033
 U 1 1 52F05898
@@
 $EndComp
 $Comp
-L +VCC #PWR034
-U 1 1 56468065
-P 11750 6175
-F 0 "#PWR034" H 11750 6275 30  0001 C CNN
-F 1 "+VCC" H 11725 6450 60  0000 C CNN
-F 2 "~" H 11750 6175 60  0000 C CNN
-F 3 "~" H 11750 6175 60  0000 C CNN
-	1    11750 6175
-	1    0    0    -1
-$EndComp
-$Comp
-L -VCC #PWR035
-U 1 1 56468A66
-P 11750 6975
-F 0 "#PWR035" H 11750 7075 30  0001 C CNN
-F 1 "-VCC" H 11725 7250 60  0000 C CNN
-F 2 "~" H 11750 6975 60  0000 C CNN
-F 3 "~" H 11750 6975 60  0000 C CNN
-	1    11750 6975
-	-1   0    0    1
-$EndComp
-$Comp
-L TL072- U4
-U 2 1 56468EEF
-P 15600 6575
-F 0 "U4" H 15550 6775 60  0000 L CNN
-F 1 "TL072-" H 15550 6325 60  0000 L CNN
-F 2 "MyModules:TSSOP8-JRL" H 15600 6575 60  0001 C CNN
-F 3 "" H 15600 6575 60  0000 C CNN
-	2    15600 6575
-	1    0    0    -1
-$EndComp
-$Comp
-L LM13700 U5
+L LM13700 U4
 U 1 1 56468C7F
 P 9100 2175
-F 0 "U5" H 9200 1975 60  0000 C CNN
+F 0 "U4" H 9200 1975 60  0000 C CNN
 F 1 "LM13700" H 9000 2175 60  0000 C CNN
 F 2 "MyModules:SOIC16-12-JRL" H 9100 2175 60  0001 C CNN
@@
 $EndComp
 $Comp
-L LM13700 U5
+L LM13700 U4
 U 2 1 56469641
 P 18050 6675
-F 0 "U5" H 18150 6475 60  0000 C CNN
+F 0 "U4" H 18150 6475 60  0000 C CNN
 F 1 "LM13700" H 17950 6675 60  0000 C CNN
 F 2 "MyModules:SOIC16-12-JRL" H 18050 6675 60  0001 C CNN
@@
 	1    0    0    -1
 $EndComp
+$Comp
+L TL074- U2
+U 1 1 564B6AE3
+P 4350 6575
+F 0 "U2" H 4400 6775 60  0000 C CNN
+F 1 "TL074-" H 4500 6375 50  0000 C CNN
+F 2 "Housings_SSOP:TSSOP-14_4.4x5mm_Pitch0.65mm" H 4350 6575 60  0001 C CNN
+F 3 "" H 4350 6575 60  0000 C CNN
+	1    4350 6575
+	1    0    0    -1
+$EndComp
+$Comp
+L TL074- U2
+U 2 1 564B6F9A
+P 11850 6575
+F 0 "U2" H 11900 6775 60  0000 C CNN
+F 1 "TL074-" H 12000 6375 50  0000 C CNN
+F 2 "Housings_SSOP:TSSOP-14_4.4x5mm_Pitch0.65mm" H 11850 6575 60  0001 C CNN
+F 3 "" H 11850 6575 60  0000 C CNN
+	2    11850 6575
+	1    0    0    -1
+$EndComp
+$Comp
+L TL074- U2
+U 3 1 564B7368
+P 15600 6575
+F 0 "U2" H 15650 6775 60  0000 C CNN
+F 1 "TL074-" H 15750 6375 50  0000 C CNN
+F 2 "Housings_SSOP:TSSOP-14_4.4x5mm_Pitch0.65mm" H 15600 6575 60  0001 C CNN
+F 3 "" H 15600 6575 60  0000 C CNN
+	3    15600 6575
+	1    0    0    -1
+$EndComp
+$Comp
+L TL074- U2
+U 4 1 564B78BD
+P 8100 6575
+F 0 "U2" H 8150 6775 60  0000 C CNN
+F 1 "TL074-" H 8250 6375 50  0000 C CNN
+F 2 "Housings_SSOP:TSSOP-14_4.4x5mm_Pitch0.65mm" H 8100 6575 60  0001 C CNN
+F 3 "" H 8100 6575 60  0000 C CNN
+	4    8100 6575
+	1    0    0    -1
+$EndComp

Commit message: bah, more hopelessness
Connections:
- net GND: now also U5.3 (+); no longer U5.5 (+)
- net VCA_OUT: now also U5.6 (-), U5.7; no longer U5.1, U5.2 (-)
- net at C1.2, Q1.6 (C1), R1.1: now also U5.2 (-); no longer U5.6 (-)
- net at C1.1, R2.2: now also U5.1; no longer U5.7
- net at C6.1, R26.1, U4.5: now also U5.5 (+); no longer U5.3 (+)
Other:
- moved on the sheet: U5A, U5B
Changed lines of the file:
@@
 L TL072- U5
 U 2 1 52F068F8
-P 16800 3375
-F 0 "U5" H 16750 3575 60  0000 L CNN
-F 1 "TL072-" H 16750 3125 60  0000 L CNN
-F 2 "MyModules:TSSOP8-JRL" H 16800 3375 60  0001 C CNN
-F 3 "~" H 16800 3375 60  0000 C CNN
-	2    16800 3375
+P 11100 2075
+F 0 "U5" H 11050 2275 60  0000 L CNN
+F 1 "TL072-" H 11050 1825 60  0000 L CNN
+F 2 "MyModules:TSSOP8-JRL" H 11100 2075 60  0001 C CNN
+F 3 "~" H 11100 2075 60  0000 C CNN
+	2    11100 2075
 	1    0    0    -1
 $EndComp
@@
 L TL072- U5
 U 1 1 52F070C4
-P 11100 2075
-F 0 "U5" H 11050 2275 60  0000 L CNN
-F 1 "TL072-" H 11050 1825 60  0000 L CNN
-F 2 "MyModules:TSSOP8-JRL" H 11100 2075 60  0001 C CNN
-F 3 "~" H 11100 2075 60  0000 C CNN
-	1    11100 2075
+P 16800 3375
+F 0 "U5" H 16750 3575 60  0000 L CNN
+F 1 "TL072-" H 16750 3125 60  0000 L CNN
+F 2 "MyModules:TSSOP8-JRL" H 16800 3375 60  0001 C CNN
+F 3 "~" H 16800 3375 60  0000 C CNN
+	1    16800 3375
 	1    0    0    -1
 $EndComp
@@
 L +VCC #PWR025
 U 1 1 52F070CA
-P 11000 1675
-F 0 "#PWR025" H 11000 1775 30  0001 C CNN
-F 1 "+VCC" H 10975 1950 60  0000 C CNN
-F 2 "~" H 11000 1675 60  0000 C CNN
-F 3 "~" H 11000 1675 60  0000 C CNN
-	1    11000 1675
+P 16700 2975
+F 0 "#PWR025" H 16700 3075 30  0001 C CNN
+F 1 "+VCC" H 16675 3250 60  0000 C CNN
+F 2 "~" H 16700 2975 60  0000 C CNN
+F 3 "~" H 16700 2975 60  0000 C CNN
+	1    16700 2975
 	1    0    0    -1
 $EndComp
@@
 L -VCC #PWR026
 U 1 1 52F070D0
-P 11000 2475
-F 0 "#PWR026" H 11000 2575 30  0001 C CNN
-F 1 "-VCC" H 10975 2750 60  0000 C CNN
-F 2 "~" H 11000 2475 60  0000 C CNN
-F 3 "~" H 11000 2475 60  0000 C CNN
-	1    11000 2475
+P 16700 3775
+F 0 "#PWR026" H 16700 3875 30  0001 C CNN
+F 1 "-VCC" H 16675 4050 60  0000 C CNN
+F 2 "~" H 16700 3775 60  0000 C CNN
+F 3 "~" H 16700 3775 60  0000 C CNN
+	1    16700 3775
 	-1   0    0    1
 $EndComp
